File: kicad/esp32-calendar/esp32-calendar.kicad_sch (KiCad schematic)
At the start: 9 parts, among them SW1 SW_Push_SPDT

Commit message: added fritzing schematics, updated schematics
Parts:
- C1: value 10uF_16V -> 0.1uF_16V
- R3: value 470k -> 780K
Changed lines of the file:
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@@
 			)
 		)
-		(property "Value" "470k"
+		(property "Value" "780K"
 			(at 90.17 118.11 0)
 			(effects
@@
 			)
 		)
-		(property "Value" "10uF_16V"
+		(property "Value" "0.1uF_16V"
 			(at 212.09 91.44 0)
 			(effects
